File: Kicad/X1_SD.kicad_pcb (KiCad board)
At the start: 2 copper layers, 137 x 140.7 mm, 40 parts, among them J1 Conn_02x22_Row_Letter_First, J2 Micro_SD_Card_Kit, J3 MicroSD Card Adapter, J4 Conn_02x22_Odd_Even, J5 Conn_02x25_Odd_Even, J6 Conn_01x02, U1 74LS04, U10 74LS139, U11 74LS541, U12 8255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

Commit message: Add files via upload
Parts:
- J1: value Conn_02x22_Row_Letter_First -> for Card-Slot
- J4: value Conn_02x22_Odd_Even -> for CZ-800
- J5: value Conn_02x25_Odd_Even -> for CZ-801
- J6: value Conn_01x02 -> for CZ-801
- moved J5 2.54 mm to (61.3, 74.2)
Connections:
- J4 pad 10: GND -> /D6
- J4 pad 11: /D7 -> /A15
- J4 pad 12: /A15 -> /D7
- J4 pad 13: /phi -> /A14
- J4 pad 14: /A14 -> /phi
- J4 pad 15: /~M1 -> /A13
- J4 pad 16: /A13 -> /~M1
- J4 pad 17: /~WR -> /A12
- J4 pad 18: /A12 -> /~WR
- J4 pad 19: /~RD -> /A11
- J4 pad 20: /A11 -> /~RD
- J4 pad 21: /~IOREQ -> /A10
- J4 pad 22: /A10 -> /~IOREQ
- J4 pad 23: /~MREQ -> /A9
- J4 pad 24: /A9 -> /~MREQ
- J4 pad 25: GND -> /A8
- J4 pad 26: /A8 -> GND
- J4 pad 27: /~HALT -> /A7
- J4 pad 28: /A7 -> /~HALT
- J4 pad 29: /IE1 -> /A6
- J4 pad 3: /D3 -> /D2
- J4 pad 30: /A6 -> /IE1
- J4 pad 31: /IE0 -> /A5
- J4 pad 32: /A5 -> /IE0
- J4 pad 33: /RESET -> /A4
- J4 pad 34: /A4 -> /RESET
- J4 pad 35: /~EXIO -> /A3
- J4 pad 36: /A3 -> /~EXIO
- J4 pad 37: /~EXINT -> /A2
- J4 pad 38: /A2 -> /~EXINT
- J4 pad 39: /~EXWAIT -> /A1
- J4 pad 4: /D2 -> /D3
- J4 pad 40: /A1 -> /~EXWAIT
- J4 pad 41: /~MNI -> /A0
- J4 pad 42: /A0 -> /~MNI
- J4 pad 5: /D4 -> /D1
- J4 pad 6: /D1 -> /D4
- J4 pad 7: /D5 -> /D0
- J4 pad 8: /D0 -> /D5
- J4 pad 9: /D6 -> GND
Routing:
- net /D3: track 301.5 -> 217.3 mm, vias 2 -> 1
- net /~RD: track 185.2 -> 247.5 mm, vias 4 -> 3
- net /D4: track 245.1 -> 204.4 mm, vias 2 -> 0
- net /A1: track 190.1 -> 218.0 mm, vias 2 -> 0
- net +5V: track 490.2 -> 509.6 mm, vias 2 -> 1
- net /~MNI: track 89.8 -> 71.7 mm, vias 2 -> 1
- net /D1: track 223.6 -> 209.4 mm
- net /CS: track 70.7 -> 56.9 mm, vias 1 -> 0
- net /A6: track 107.0 -> 119.6 mm, vias 1 -> 3
- net /MISO: track 63.1 -> 75.1 mm
- net /~M1: track 41.5 -> 53.3 mm
- net /A0: track 187.2 -> 198.1 mm, vias 1 -> 0
- net /MOSI: track 59.5 -> 70.3 mm, vias 0 -> 1
- net /A15: track 59.5 -> 48.8 mm
- net /A8: track 126.0 -> 136.5 mm, vias 2 -> 4
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Other:
- board text added: "X1_SD Rev1.3"
- board text removed: "X1_SD Rev1.2"
